Commit message: tried adding slam

File: description/robot_core.xacro (robot description, xacro)
@@ -20,4 +20,11 @@
     <link name="base_link">
     </link>
+    <!--  Base Footprint-->
+    <joint name="base_footprint" type="fixed">
+        <parent link="base_link"/>
+        <child link="base_footprint"/>
+        <origin xyz="0 0 0" rpy="0 0 0"/>
+    </joint>
+    <link name="base_footprint"></link>
     <!-- Chassis Link-->
     <joint name="chassis_joint" type="fixed">
